Commit message: Add files via upload

File: urdf/franka_description/robots/spoon_franka.urdf (robot description, URDF)
Before this commit: robot panda, 11 links, 10 joints
Links:
- link panda_hand: geometry collision mesh filename=meshes/collision/combine_hand.obj; visual mesh filename=meshes/visual/spoon_hand.obj
